File: pcb/BS_Power/BS_Power.kicad_sch (KiCad schematic)
At the start: 7 parts, among them J1 Barrel_Jack_Switch, J2 POWER, J3 Conn_02x07_Odd_Even, J4 Conn_01x02

Commit message: Before 5V regulator replacement
Parts:
- removed J4: Conn_01x02, Parts:MOLEX_430450212, symbol Connector_Generic:Conn_01x02
- added J4: 436500400, MOLEX_436500400, symbol 436500400:436500400
- J2: LCSC Part (none) -> C9144
- J3: LCSC Part (none) -> C383616
Connections:
- net +12V: now also J4.2; no longer J2.3 (Pin_3)
- net +3V3: now also J4.4; no longer J2.7 (Pin_7)
- net +5V: now also J4.3; no longer J2.5 (Pin_5)
- net GND: now also J4.1

Commit message: BS_Power updates
Parts:
- J3: LCSC Part C383616 -> C146614
- J4: footprint MOLEX_436500400 -> Parts:MOLEX_436500400

Commit message: BSPower V2
Parts:
- D1: value SMAJ16A -> SMAJ15CA; LCSC Part C908770 -> C353477
Changed lines of the file:
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@@
       (effects (font (size 1.27 1.27)) (justify left))
     )
-    (property "Value" "SMAJ16A" (id 1) (at 52.07 68.58 90)
+    (property "Value" "SMAJ15CA" (id 1) (at 52.07 68.58 90)
       (effects (font (size 1.27 1.27)) (justify left))
     )
@@
       (effects (font (size 1.27 1.27)) hide)
     )
-    (property "LCSC Part" "C908770" (id 4) (at 50.8 66.04 90)
+    (property "LCSC Part" "C353477" (id 4) (at 50.8 66.04 90)
       (effects (font (size 1.27 1.27)) hide)
     )
@@
     )
     (path "/d200cae5-4ea1-4a26-90db-fb0f7da5ff0c"
-      (reference "D1") (unit 1) (value "SMAJ16A") (footprint "Diode_SMD:D_SMA")
+      (reference "D1") (unit 1) (value "SMAJ15CA") (footprint "Diode_SMD:D_SMA")
     )
     (path "/1989359f-ada5-4906-a23b-5c103295523a"
