File: pcb/BS_Power/PowerPS.kicad_sch (KiCad schematic)
At the start: 10 parts

Commit message: BS_Power updates
Parts:
- L3: footprint Beefy:L_4.45x4.06 -> Beefy:L_4.1x4.5; LCSC Part C844980 -> C2847469
Changed lines of the file:
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@@
     (property "Reference" "L3" (id 0) (at 111.76 33.02 90))
     (property "Value" "2.2uH" (id 1) (at 111.76 38.1 90))
-    (property "Footprint" "Beefy:L_4.45x4.06" (id 2) (at 111.76 35.56 0)
+    (property "Footprint" "Beefy:L_4.1x4.5" (id 2) (at 111.76 35.56 0)
       (effects (font (size 1.27 1.27)) hide)
     )
@@
       (effects (font (size 1.27 1.27)) hide)
     )
-    (property "LCSC Part" "C844980" (id 4) (at 111.76 35.56 90)
+    (property "LCSC Part" "C2847469" (id 4) (at 111.76 35.56 90)
       (effects (font (size 1.27 1.27)) hide)
     )

Commit message: BSPower V2
Connections:
- net +5V: now also C18.1, PS3.10 (AVIN)
Changed lines of the file:
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@@
   (junction (at 72.39 35.56) (diameter 0) (color 0 0 0 0)
+  )
+  (junction (at 50.8 38.1) (diameter 0) (color 0 0 0 0)
   )
   (junction (at 105.41 38.1) (diameter 0) (color 0 0 0 0)
@@
   )
   (junction (at 120.65 35.56) (diameter 0) (color 0 0 0 0)
+  )
+  (junction (at 50.8 35.56) (diameter 0) (color 0 0 0 0)
   )
   (junction (at 43.18 59.69) (diameter 0) (color 0 0 0 0)
@@
     (stroke (width 0) (type default) (color 0 0 0 0))
   )
+  (wire (pts (xy 50.8 35.56) (xy 72.39 35.56))
+    (stroke (width 0) (type default) (color 0 0 0 0))
+  )
   (wire (pts (xy 104.14 60.96) (xy 107.95 60.96))
     (stroke (width 0) (type default) (color 0 0 0 0))
@@
     (stroke (width 0) (type default) (color 0 0 0 0))
   )
-  (wire (pts (xy 43.18 35.56) (xy 72.39 35.56))
+  (wire (pts (xy 43.18 35.56) (xy 50.8 35.56))
     (stroke (width 0) (type default) (color 0 0 0 0))
   )
@@
     (stroke (width 0) (type default) (color 0 0 0 0))
   )
+  (wire (pts (xy 50.8 35.56) (xy 50.8 38.1))
+    (stroke (width 0) (type default) (color 0 0 0 0))
+  )
